Commit message: update

File: gh360/urdf/gh360.urdf (robot description, URDF)
Before this commit: robot multipleshapes, 12 links, 11 joints
Links:
- added link eef; visual sphere radius=0.01
Joints:
- removed joint lowerarm_eef_connect
- added joint lowerarm_tool_connect: type fixed, parent lowerarm2, child hook, origin xyz=0.00 -0.037 -0.001 rpy=3.1415 1.5708 0
- added joint tool_eef_connect: type fixed, parent hook, child eef, origin xyz=0.0 0.05 0.0 rpy=0.0 0.0 0
- joint base_joint: origin xyz=0.0 0 0.5 rpy=1.571 0 1.571 -> xyz=-0.66 0.0 1.112 rpy=1.571 0 1.571

Commit message: update

File: gh360/urdf/gh360.urdf (robot description, URDF)
Before this commit: robot multipleshapes, 13 links, 12 joints
Joints:
- joint base_joint: origin xyz=-0.66 0.0 1.112 rpy=1.571 0 1.571 -> xyz=-0.66 0.0 1.242 rpy=1.571 0 1.571

Commit message: feat: robosuite spacemouse teleop

File: gh360/urdf/gh360.urdf (robot description, URDF)
Before this commit: robot multipleshapes, 13 links, 12 joints
Joints:
- joint base_joint: origin xyz=-0.66 0.0 1.242 rpy=1.571 0 1.571 -> xyz=-0.26 0.0 0.330 rpy=1.571 0 1.571
